Commit message: Update fetch+leap urdf and remove the copied leap meshes.

File: fetch_description/robots/fetch_leap.urdf (robot description, URDF)
Before this commit: robot fetch, 42 links, 41 joints
Links:
- link dip: mass 0.005 -> 0.037; geometry collision mesh filename=package://leap_description/meshes/collisions/box_dip.stl; visual mesh filename=package://leap_description/meshes/dip.stl
- link dip_2: mass 0.005 -> 0.037; geometry collision mesh filename=package://leap_description/meshes/collisions/box_dip.stl; visual mesh filename=package://leap_description/meshes/dip.stl
- link dip_3: mass 0.005 -> 0.037; geometry collision mesh filename=package://leap_description/meshes/collisions/box_dip.stl; visual mesh filename=package://leap_description/meshes/dip.stl
- link fingertip: mass 0.005 -> 0.016; geometry collision mesh filename=package://leap_description/meshes/collisions/box_fingertip.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; visual mesh filename=package://leap_description/meshes/fingertip.stl
- link fingertip_2: mass 0.005 -> 0.016; geometry collision mesh filename=package://leap_description/meshes/collisions/box_fingertip.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; visual mesh filename=package://leap_description/meshes/fingertip.stl
- link fingertip_3: mass 0.005 -> 0.016; geometry collision mesh filename=package://leap_description/meshes/collisions/box_fingertip.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; visual mesh filename=package://leap_description/meshes/fingertip.stl
- link mcp_joint: mass 0.005 -> 0.044; geometry collision mesh filename=package://leap_description/meshes/collisions/box_mcp_joint.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; visual mesh filename=package://leap_description/meshes/mcp_joint.stl
- link mcp_joint_2: mass 0.005 -> 0.044; geometry collision mesh filename=package://leap_description/meshes/collisions/box_mcp_joint.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; visual mesh filename=package://leap_description/meshes/mcp_joint.stl
- link mcp_joint_3: mass 0.005 -> 0.044; geometry collision mesh filename=package://leap_description/meshes/collisions/box_mcp_joint.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; visual mesh filename=package://leap_description/meshes/mcp_joint.stl
- link palm_lower: mass 0.826 -> 0.385; geometry collision mesh filename=package://leap_description/meshes/collisions/box_palm_lower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; visual mesh filename=package://leap_description/meshes/palm_lower_fetch.stl
- link pip: mass 0.005 -> 0.032; geometry collision mesh filename=package://leap_description/meshes/collisions/box_pip.stl; visual mesh filename=package://leap_description/meshes/pip.stl
- link pip_2: mass 0.005 -> 0.032; geometry collision mesh filename=package://leap_description/meshes/collisions/box_pip.stl; visual mesh filename=package://leap_description/meshes/pip.stl
- link pip_3: mass 0.005 -> 0.032; geometry collision mesh filename=package://leap_description/meshes/collisions/box_pip.stl; visual mesh filename=package://leap_description/meshes/pip.stl
- link pip_4: mass 0.005 -> 0.032; geometry collision mesh filename=package://leap_description/meshes/collisions/box_pip.stl; visual mesh filename=package://leap_description/meshes/pip.stl
- link thumb_dip: mass 0.005 -> 0.038; geometry collision mesh filename=package://leap_description/meshes/collisions/box_thumb_dip.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; visual mesh filename=package://leap_description/meshes/thumb_dip.stl
- link thumb_fingertip: mass 0.005 -> 0.049; geometry collision mesh filename=package://leap_description/meshes/collisions/box_thumb_fing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; visual mesh filename=package://leap_description/meshes/thumb_fingertip.stl
- link thumb_pip: mass 0.005 -> 0.003; geometry collision mesh filename=package://leap_description/meshes/collisions/box_thumb_pip.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; visual mesh filename=package://leap_description/meshes/thumb_pip.stl
Joints:
- removed joint ati_to_leap_hand
- added joint ati_to_leap: type fixed, parent ati_link, child palm_lower, origin xyz=0.01328 0.03674 0.06010 rpy=0 -1.5708 0
